Commit message: T-1 day

File: src/adele_urdf_2/urdf/adele_urdf_2.urdf (robot description, URDF)
Before this commit: robot adele_urdf_2, 7 links, 6 joints
Links:
- added link dummy
Joints:
- added joint dummy_joint: type fixed, parent dummy, child base_link
- joint Joint_1: limit lower=-2 upper=2 effort=0 velocity=125.7 -> lower=-2 upper=2 effort=0.1 velocity=125.7
- joint Joint_2: limit lower=-1.57 upper=1.57 effort=0 velocity=125.7 -> lower=-1.57 upper=1.57 effort=0.1 velocity=125.7
- joint Joint_3: limit lower=-1.57 upper=1.57 effort=0 velocity=125.7 -> lower=-1.57 upper=1.57 effort=0.1 velocity=125.7
- joint Joint_4: limit lower=-1.57 upper=1.57 effort=0 velocity=125.7 -> lower=-1.57 upper=1.57 effort=0.1 velocity=125.7
- joint Joint_5: limit lower=-1.57 upper=1.57 effort=0 velocity=125.7 -> lower=-1.57 upper=1.57 effort=0.1 velocity=125.7
- joint Joint_6: axis -1 0 0 -> 1 0 0; limit lower=-0.785398 upper=0.785398 effort=0 velocity=125.7 -> lower=-0.785398 upper=0.785398 effort=0.1 velocity=125.7

Commit message: Update

File: src/adele_urdf_2/urdf/adele_urdf_2.urdf (robot description, URDF)
Before this commit: robot adele_urdf_2, 8 links, 7 joints
Joints:
- joint Joint_5: limit lower=-1.57 upper=1.57 effort=0.1 velocity=125.7 -> lower=-0.785398 upper=0.785398 effort=0.1 velocity=125.7
- joint Joint_6: limit lower=-0.785398 upper=0.785398 effort=0.1 velocity=125.7 -> lower=-1.57 upper=1.57 effort=0.1 velocity=125.7

Commit message: updated moveit package

File: src/adele_urdf_2/urdf/adele_urdf_2.urdf (robot description, URDF)
Before this commit: robot adele_urdf_2, 8 links, 7 joints
Joints:
- joint Joint_1: limit lower=-2 upper=2 effort=0.1 velocity=125.7 -> lower=-2.0 upper=2.0 effort=0.1 velocity=125.7

Commit message: Revert "Update"
This reverts commit 994342cbde1b499da19b56b78d9710148e3cdba8.

File: src/adele_urdf_2/urdf/adele_urdf_2.urdf (robot description, URDF)
Before this commit: robot adele_urdf_2, 8 links, 7 joints
Joints:
- joint Joint_5: limit lower=-0.785398 upper=0.785398 effort=0.1 velocity=125.7 -> lower=-1.57 upper=1.57 effort=0.1 velocity=125.7
- joint Joint_6: limit lower=-1.57 upper=1.57 effort=0.1 velocity=125.7 -> lower=-0.785398 upper=0.785398 effort=0.1 velocity=125.7

Commit message: Revert "updated moveit package"
This reverts commit 41f08bf72e1689826443133b34101b776144a05f.

File: src/adele_urdf_2/urdf/adele_urdf_2.urdf (robot description, URDF)
Before this commit: robot adele_urdf_2, 8 links, 7 joints
Joints:
- joint Joint_1: limit lower=-2.0 upper=2.0 effort=0.1 velocity=125.7 -> lower=-2 upper=2 effort=0.1 velocity=125.7

Commit message: Updated joint limits

File: src/adele_urdf_2/urdf/adele_urdf_2.urdf (robot description, URDF)
Before this commit: robot adele_urdf_2, 8 links, 7 joints
Joints:
- joint Joint_1: limit lower=-2 upper=2 effort=0.1 velocity=125.7 -> lower=-3.1416 upper=3.1416 effort=0.1 velocity=125.7
- joint Joint_5: limit lower=-1.57 upper=1.57 effort=0.1 velocity=125.7 -> lower=-0.785398 upper=0.785398 effort=0.1 velocity=125.7
- joint Joint_6: limit lower=-0.785398 upper=0.785398 effort=0.1 velocity=125.7 -> lower=-1.57 upper=1.57 effort=0.1 velocity=125.7
